File: schema/KiCad/lampeDimmer/lampeDimmer.kicad_pcb (KiCad board)
At the start: 2 copper layers, 76.5 x 46.3 mm, 28 parts, among them J1 PICkit4, J2 USART, J3 EXT_IO, J4 EXT_PWM4B, J5 EXT_PWM4D, J6 EXT_ADC1, J7 CON_POT_SW, J8 Entrée, J9 Sortie, M1 ARDUINO_MICRO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

Commit message: ~ Mise à jours des noms de labels sur le schéma. ~ Mise à jours du PCB. ~ Mise à jours des fichiers Gerbers.
Parts:
- removed SW1: SW_ON-OFF, Connector_PinSocket_2.54mm:PinSocket_1x02_P2.54mm_Vertical
- added J10: Sortie, TerminalBlock:TerminalBlock_bornier-2_P5.08mm, F.Cu at (122.3, 99.3)
- J3: value EXT_IO -> EXT_IO-1
- J4: value EXT_PWM4B -> SW_ON-OFF
- J5: value EXT_PWM4D -> EXT_PWM4B
- J6: value EXT_ADC1 -> EXT_PWM4D
- J7: value CON_POT_SW -> EXT_ADC1; footprint Connector_PinSocket_2.54mm:PinSocket_1x05_P2.54mm_Vertical -> Connector_PinSocket_2.54mm:PinSocket_1x02_P2.54mm_Vertical
- J8: value Entrée -> CON_POT_SW; footprint TerminalBlock:TerminalBlock_bornier-2_P5.08mm -> Connector_PinSocket_2.54mm:PinSocket_1x05_P2.54mm_Vertical
- J9: value Sortie -> Entrée
- moved J7 49.5 mm to (183.7, 119.5), turned to 90 degrees
- moved J4 26.7 mm to (137.2, 117.1)
- moved J6 21.5 mm to (162.2, 119.6)
- moved J8 21.2 mm to (139.3, 97.6), turned to 0 degrees
- moved J9 11.0 mm to (122.3, 110.3)
- moved J5 6.88 mm to (162.1, 126.5)
Connections:
- net /EXT_IO renamed /EXT_IO-1
- J4 pad 2: /EXT_OC4B -> /SW_ON-OFF
- J5 pad 2: /EXT_OC4D -> /EXT_OC4B
- J6 pad 2: /EXT_ADC1 -> /EXT_OC4D
- J7 pad 1: +5V -> GND
- J7 pad 2: /POT_ADC -> /EXT_ADC1
- J8 pad 1: +24V -> +5V
- J8 pad 2: GND -> /POT_ADC
- J9 pad 1: /SORTIE -> +24V
- J9 pad 2: +24V -> GND
- M1 pad 34: Net-(M1-Pad34) -> /SW_ON-OFF
Routing:
- net Net-(M1-Pad34): track 20.9 -> 0.00 mm, vias 2 -> 0
- net /SW_ON-OFF: track 0.00 -> 20.9 mm, vias 0 -> 2
